File: KiCad/Architectural scheme.sch (KiCad schematic (older format))
At the start: 5 parts

Commit message: Last commit
Parts:
- u: value ESP-01 -> ESP8266-01
Connections:
- net +3V3: now also u.3 (CH_PD)
Other:
- note removed: "Figura 2"
Changed lines of the file:
@@
 $EndDescr
-$Comp
-L ESP8266:ESP-01v090 u
-U 1 1 61BD342E
-P 2250 4850
-F 0 "u" H 2250 5365 50  0001 C CNN
-F 1 "ESP-01" H 2250 5274 50  0000 C CNB
-F 2 "" H 2250 4850 50  0001 C CNN
-F 3 "http://l0l.org.uk/2014/12/esp8266-modules-hardware-guide-gotta-catch-em-all/" H 2250 4850 50  0001 C CNN
-	1    2250 4850
-	1    0    0    -1
-$EndComp
 $Comp
 L Sensor_Motion:MPU-6050 U?
@@
 Wire Wire Line
 	1150 850  5350 850
-Wire Wire Line
-	1300 4700 1300 3800
 Wire Wire Line
 	1300 3800 7550 3800
@@
 Text Notes 5000 3750 1    50   ~ 0
 USART3_DEBUG_RX
-Text Notes 10900 6050 1    138  ~ 0
-Figura 2
+Wire Wire Line
+	1300 4700 1300 3800
+$Comp
+L ESP8266:ESP-01v090 u
+U 1 1 61BD342E
+P 2250 4850
+F 0 "u" H 2250 5365 50  0001 C CNN
+F 1 "ESP8266-01" H 2250 5274 50  0000 C CNB
+F 2 "" H 2250 4850 50  0001 C CNN
+F 3 "http://l0l.org.uk/2014/12/esp8266-modules-hardware-guide-gotta-catch-em-all/" H 2250 4850 50  0001 C CNN
+	1    2250 4850
+	1    0    0    -1
+$EndComp
+$Comp
+L power:+3.3V #PWR?
+U 1 1 61F7D275
+P 1050 4800
+F 0 "#PWR?" H 1050 4650 50  0001 C CNN
+F 1 "+3.3V" H 1065 4973 50  0000 C CNN
+F 2 "" H 1050 4800 50  0001 C CNN
+F 3 "" H 1050 4800 50  0001 C CNN
+	1    1050 4800
+	0    -1   -1   0
+$EndComp
+Wire Wire Line
+	1300 4800 1050 4800
 $EndSCHEMATC
